File: recruitment.kicad_sch (KiCad schematic)
At the start: 12 parts, among them J1 Conn_01x02_Pin, K1 Relay_SPST-NO, U1 OKI-78SR-5_1.5-W36-C

Commit message: wired pcb
Parts:
- added J2: Conn_01x02_Pin, symbol Connector:Conn_01x02_Pin
- K1: footprint LED_THT:LED_D3.0mm -> Relay_THT:Relay_SPST_Finder_32.21-x300
Connections:
- net GND: now also J2.2 (Pin_2)
- net +36V renamed 36V
- net 36V: now also J2.1 (Pin_1)
- net 3.3V renamed VCC
- net 9-17V: no longer names the net of J1.1 (Pin_1), R1.1, U1.1 (IN)
Changed lines of the file:
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@@
+	)
+	(junction
+		(at 118.11 57.15)
+		(diameter 0)
+		(color 0 0 0 0)
 	)
 	(junction
@@
 	(wire
 		(pts
+			(xy 118.11 57.15) (xy 118.11 59.69)
+		)
+		(stroke
+			(width 0)
+			(type default)
+		)
+	)
+	(wire
+		(pts
 			(xy 115.57 80.01) (xy 115.57 86.36)
 		)
@@
 	(wire
 		(pts
+			(xy 90.17 57.15) (xy 118.11 57.15)
+		)
+		(stroke
+			(width 0)
+			(type default)
+		)
+	)
+	(wire
+		(pts
 			(xy 90.17 80.01) (xy 115.57 80.01)
 		)
@@
 	(wire
 		(pts
-			(xy 118.11 54.61) (xy 118.11 59.69)
+			(xy 118.11 54.61) (xy 118.11 57.15)
 		)
 		(stroke
@@
 	(wire
 		(pts
-			(xy 92.71 25.4) (xy 92.71 39.37)
+			(xy 92.71 21.59) (xy 92.71 39.37)
 		)
 		(stroke
@@
 		(pts
 			(xy 90.17 102.87) (xy 113.03 102.87)
+		)
+		(stroke
+			(width 0)
+			(type default)
+		)
+	)
+	(wire
+		(pts
+			(xy 90.17 21.59) (xy 90.17 57.15)
 		)
 		(stroke
@@
 		)
 	)
-	(label "RL1+"
-		(at 196.85 64.77 0)
-		(effects
-			(font
-				(size 1.27 1.27)
-			)
-			(justify left bottom)
-		)
-	)
-	(label "9-17V"
-		(at 60.96 80.01 0)
-		(effects
-			(font
-				(size 1.27 1.27)
-			)
-			(justify left bottom)
-		)
-	)
 	(label "5V"
 		(at 83.82 80.01 0)
@@
 		)
 	)
-	(label "3.3V"
+	(label "VCC"
 		(at 171.45 69.85 0)
 		(effects
@@
 		)
 	)
-	(label "3.3V"
+	(label "VCC"
 		(at 134.62 69.85 0)
 		(effects
@@
 		)
 	)
-	(label "RL1-"
-		(at 191.77 58.42 0)
-		(effects
-			(font
-				(size 1.27 1.27)
-			)
-			(justify left bottom)
-		)
-	)
 	(label "GND"
 		(at 185.42 102.87 0)
@@
 		)
 	)
-	(label "VCC_H"
+	(label "VCC"
 		(at 201.93 78.74 0)
 		(effects
@@
 			)
 		)
-		(property "Footprint" "LED_THT:LED_D3.0mm"
+		(property "Footprint" "Relay_THT:Relay_SPST_Finder_32.21-x300"
 			(at 172.72 35.56 0)
 			(effects
@@
 				(path "/bdc7face-9f7c-4701-80bb-4cc144448db1"
 					(reference "K1")
+					(unit 1)
+				)
+			)
+		)
+	)
+	(symbol
+		(lib_id "Connector:Conn_01x02_Pin")
+		(at 92.71 16.51 270)
+		(unit 1)
+		(exclude_from_sim no)
+		(in_bom yes)
+		(on_board yes)
+		(dnp no)
+		(fields_autoplaced yes)
+		(property "Reference" "J2"
+			(at 93.98 15.8749 90)
+			(effects
+				(font
+					(size 1.27 1.27)
+				)
+				(justify left)
+			)
+		)
+		(property "Value" "Conn_01x02_Pin"
+			(at 93.98 18.4149 90)
+			(effects
+				(font
+					(size 1.27 1.27)
+				)
+				(justify left)
+			)
+		)
+		(property "Footprint" ""
+			(at 92.71 16.51 0)
+			(effects
+				(font
+					(size 1.27 1.27)
+				)
+				(hide yes)
+			)
+		)
+		(property "Datasheet" "~"
+			(at 92.71 16.51 0)
+			(effects
+				(font
+					(size 1.27 1.27)
+				)
+				(hide yes)
+			)
+		)
+		(property "Description" "Generic connector, single row, 01x02, script generated"
+			(at 92.71 16.51 0)
+			(effects
+				(font
+					(size 1.27 1.27)
+				)
+				(hide yes)
+			)
+		)
+		(pin "1"
+		)
+		(pin "2"
+		)
+		(instances
+			(project ""
+				(path "/bdc7face-9f7c-4701-80bb-4cc144448db1"
+					(reference "J2")
 					(unit 1)
 				)
@@
 					(unit 1)
 				)
-			)
-		)
-	)
-	(symbol
-		(lib_id "power:+36V")
-		(at 92.71 25.4 0)
-		(unit 1)
-		(exclude_from_sim no)
-		(in_bom yes)
-		(on_board yes)
-		(dnp no)
-		(fields_autoplaced yes)
-		(property "Reference" "#PWR02"
-			(at 92.71 29.21 0)
-			(effects
-				(font
-					(size 1.27 1.27)
-				)
-				(hide yes)
-			)
-		)
-		(property "Value" "+36V"
-			(at 92.71 20.32 0)
-			(effects
-				(font
-					(size 1.27 1.27)
-				)
-			)
-		)
-		(property "Footprint" ""
-			(at 92.71 25.4 0)
-			(effects
-				(font
-					(size 1.27 1.27)
-				)
-				(hide yes)
-			)
-		)
-		(property "Datasheet" ""
-			(at 92.71 25.4 0)
-			(effects
-				(font
-					(size 1.27 1.27)
-				)
-				(hide yes)
-			)
-		)
-		(property "Description" "Power symbol creates a global label with name \"+36V\""
-			(at 92.71 25.4 0)
-			(effects
-				(font
-					(size 1.27 1.27)
-				)
-				(hide yes)
-			)
-		)
-		(pin "1"
-		)
-		(instances
-			(project ""
-				(path "/bdc7face-9f7c-4701-80bb-4cc144448db1"
-					(reference "#PWR02")
-					(unit 1)
-				)
