File: monitor.kicad_sch (KiCad schematic)
At the start: 5 parts, among them K2 Relay_SPDT, SW2 SW_Wuerth_450301014042, U2 LM397, U3 SCR

Commit message: wired pcb
Other:
- note added: "U2"
Changed lines of the file:
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@@
 	(generator_version "9.0")
 	(paper "A4")
+	(text "U2\n"
+		(exclude_from_sim no)
+		(at 155.956 87.63 0)
+		(effects
+			(font
+				(size 1.27 1.27)
+			)
+		)
+	)
 	(text "Monostable"
 		(exclude_from_sim no)
